File: KiCadCircuit/Circuit/Circuit.kicad_sch (KiCad schematic)
At the start: 14 parts, among them M1 Motor_DC, M2 Motor_DC, M3 Motor_DC, M4 Motor_DC, Q1 IRLZ44N, Q2 IRLZ44N, Q3 IRLZ44N, Q4 IRLZ44N, U1 ESP32-WROOM-32U

Commit message: Diodes added for motors
Parts:
- added D1, D2, D3, D4: D, symbol Device:D
Connections:
- net at M4.1 (+), Q4.2 (D): now also D1.1 (K)
- net at M3.1 (+), Q3.2 (D): now also D2.1 (K)
- net at M1.1 (+), Q1.2 (D): now also D4.1 (K)
- net at BT1.2 (-), U1.1 (GND), U1.15 (GND)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: now also M1.2 (-), M2.2 (-), M3.2 (-), M4.2 (-), D1.2 (A), D2.2 (A), D3.2 (A), D4.2 (A)
- net at M2.1 (+), Q2.2 (D): now also D3.1 (K)
Other:
- moved on the sheet: BT1, M1, M2, M3, M4, Q1, Q2, Q3, Q4, R1, R2, R3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

Commit message: ToDoList in Readme
Parts:
- added R5, R6, R7, R8: 10k, symbol Device:R
Connections:
- net at BT1.1 (+), Q1.3 (S), Q2.3 (S)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: no longer R4.2, U1.36 (IO22)
- net at BT1.2 (-), D1.2 (A), D2.2 (A)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: now also R5.2, R6.2, R7.2, R8.2
- net at R1.2, U1.27 (IO16): now also R5.1
- net at R2.2, U1.28 (IO17): now also R6.1
- net at R3.2, U1.33 (IO21): now also R7.1
- new net: R4.2, R8.1, U1.36 (IO22)
Other:
- title: (none) -> Drone Circuit
- moved on the sheet: BT1

Commit message: KiCadCircuit finished for Drone
Parts:
- added U2: MPU-6050, Sensor_Motion:InvenSense_QFN-24_4x4mm_P0.5mm, symbol Sensor_Motion:MPU-6050
- R1, R2, R3, R4: value 1k -> 330
Connections:
- net +3.3V: now reaches BT1.1 (+), Q1.3 (S), Q2.3 (S), Q3.3 (S), Q4.3 (S)
- net +3.3V: now also U1.2 (VDD), U2.13 (VDD), U2.8 (VLOGIC)
- net at BT1.2 (-), D1.2 (A), D2.2 (A)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: now also U2.18 (GND)
- net at U1.30 (IO18): now also R3.2, R7.1
- net at U1.31 (IO19): now also R4.2, R8.1
- new net: U1.33 (IO21), U2.24 (SDA)
- new net: U1.36 (IO22), U2.23 (SCL)
Other:
- note added: "Spannungsregler bereits auf DevKit-board vorhanden"
- moved on the sheet: U1

Commit message: fixed KiCad motor falsly poled
Connections:
- net +3.3V: now also D1.1 (K), D2.1 (K), D3.1 (K), D4.1 (K), M1.1 (+), M2.1 (+), M3.1 (+), M4.1 (+); no longer Q1.3 (S), Q2.3 (S), Q3.3 (S), Q4.3 (S)
- net at BT1.2 (-), R5.2, R6.2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: now also Q1.3 (S), Q2.3 (S), Q3.3 (S), Q4.3 (S); no longer D1.2 (A), D2.2 (A), D3.2 (A), D4.2 (A), M1.2 (-), M2.2 (-), M3.2 (-), M4.2 (-)
- new net: D1.2 (A), M4.2 (-), Q4.2 (D)
- new net: D2.2 (A), M1.2 (-), Q3.2 (D)
- new net: D4.2 (A), M3.2 (-), Q1.2 (D)
- new net: D3.2 (A), M2.2 (-), Q2.2 (D)
Other:
- moved on the sheet: D1, D2, D3, D4, M1, M2, M3, M4
